File: keyboards/circuit/hardware/prod/prod.sch (EAGLE design)
At the start: 1 part, among them IC1 ATMEGA32U4

Commit message: production hw
Parts:
- added C1, C3: 1u, passives:CAP-0805
- added C2: 100n, passives:CAP-0805
- added C4, C5: 18p, passives:CAP-0805
- added D_0, D_1, D_2, D_3, D_4, D_5, D_6, D_7, D_8, D_9, D_A, D_B, D_BCK, D_C, D_CAPS, D_COLON, D_D, D_DA, D_E, D_ENTER, D_ESC, D_F, D_FN, D_G, D_GT, D_H, D_I, D_J, D_K, D_L, D_LA, D_LALT, D_LCTRL, D_LCURL, D_LSHIFT, D_LT, D_M, D_MINUS, D_N, D_O, D_OS, D_P, D_PIPE, D_PLUS, D_Q, D_QM, D_QUOTE, D_R, D_RA, D_RCURL, D_RSHIFT, D_S, D_SPACE, D_T, D_TAB, D_TILDE, D_U, D_UA, D_V, D_W, D_X, D_Y, D_Z: DIODE-BAS16L, discrete:DIODE-BAS16L
- added F1: 500m, passives:FUSE
- added ICSP: HEADER-061X6, connector:HEADER-061X6
- added J1: USB-C-2.0-CUI-UJ31-CH-G1-SMT-TR, connector-protocol:USB-C-2.0-CUI-UJ31-CH-G1-SMT-TR
- added R1, R2: 22, passives:RESISTOR-0805
- added R3, R4: 10k, passives:RESISTOR-0805
- added SW_0, SW_1, SW_2, SW_3, SW_4, SW_5, SW_6, SW_7, SW_8, SW_9, SW_A, SW_B, SW_BCK, SW_C, SW_CAPS, SW_COLON, SW_D, SW_DA, SW_E, SW_ENTER, SW_ESC, SW_F, SW_FN, SW_G, SW_GT, SW_H, SW_I, SW_J, SW_K, SW_LA, SW_LALT, SW_LCTRL, SW_LCURL, SW_LSHIFT, SW_LT, SW_M, SW_MINUS, SW_N, SW_O, SW_OS, SW_P, SW_PIPE, SW_PLUS, SW_Q, SW_QM, SW_QUOTE, SW_R, SW_RA, SW_RCURL, SW_RSHIFT, SW_S, SW_SPACE, SW_T, SW_TAB, SW_TILDE, SW_U, SW_UA, SW_V, SW_W, SW_X, SW_Y, SW_Z, S_L: SWITCH-SPSTCHERRY, passives:SWITCH-SPSTCHERRY
- added T1, T2, T3, T4: TEST-POINT, misc:TEST-POINT
- added X1: 16MHz, passives:CRYSTAL-16MHZ-CSM-3X
Connections:
- new net COL1: D_CAPS.ANODE+, D_ESC.ANODE+, D_LCTRL.ANODE+, D_LSHIFT.ANODE+, D_TAB.ANODE+, IC1.PF5(ADC5)
- new net COL10: D_9.ANODE+, D_GT.ANODE+, D_L.ANODE+, D_O.ANODE+, IC1.PD2(RX)
- new net COL11: D_0.ANODE+, D_COLON.ANODE+, D_P.ANODE+, D_QM.ANODE+, IC1.PD4(ADC8)
- new net COL12: D_LCURL.ANODE+, D_MINUS.ANODE+, D_QUOTE.ANODE+, D_RSHIFT.ANODE+, IC1.PD1(SDA)
- new net COL13: D_ENTER.ANODE+, D_PLUS.ANODE+, D_RCURL.ANODE+, IC1.PB7
- new net COL14: D_BCK.ANODE+, D_PIPE.ANODE+, IC1.PD0(SCL)
- new net COL15: D_TILDE.ANODE+, IC1.PD3(TX)
- new net COL2: D_1.ANODE+, D_A.ANODE+, D_OS.ANODE+, D_Q.ANODE+, D_Z.ANODE+, IC1.PF6(ADC6)
- new net COL3: D_2.ANODE+, D_LALT.ANODE+, D_S.ANODE+, D_W.ANODE+, D_X.ANODE+, IC1.PF7(ADC7)
- new net COL4: D_3.ANODE+, D_C.ANODE+, D_D.ANODE+, D_E.ANODE+, D_SPACE.ANODE+, IC1.PB6(ADC13)
- new net COL5: D_4.ANODE+, D_F.ANODE+, D_FN.ANODE+, D_R.ANODE+, D_V.ANODE+, IC1.PD7(ADC10)
- new net COL6: D_5.ANODE+, D_B.ANODE+, D_G.ANODE+, D_LA.ANODE+, D_T.ANODE+, IC1.PC7
- new net COL7: D_6.ANODE+, D_H.ANODE+, D_N.ANODE+, D_UA.ANODE+, D_Y.ANODE+, IC1.PC6
- new net COL8: D_7.ANODE+, D_DA.ANODE+, D_J.ANODE+, D_M.ANODE+, D_U.ANODE+, IC1.PF0(ADC0)
- new net COL9: D_8.ANODE+, D_I.ANODE+, D_K.ANODE+, D_LT.ANODE+, D_RA.ANODE+, IC1.PE6
- new net GND: C1.2, C2.2, C3.2, C4.2, C5.1, IC1.GND@15, IC1.GND@23, IC1.GND@35, IC1.GND@43, IC1.UGND, ICSP.2, J1.GND, T2.P$1, T4.P$1
- new net N$1: J1.D+, R1.1
- new net N$10: C5.2, IC1.XTAL1, X1.P$1
- new net N$101: D_LT.CATHODE-, SW_LT.P$1
- new net N$103: D_RA.CATHODE-, SW_RA.P$1
- new net N$105: D_9.CATHODE-, SW_9.P$1
- new net N$107: D_O.CATHODE-, SW_O.P$1
- new net N$109: D_L.CATHODE-, S_L.P$1
- new net N$11: D_ESC.CATHODE-, SW_ESC.P$1
- new net N$111: D_GT.CATHODE-, SW_GT.P$1
- new net N$115: D_0.CATHODE-, SW_0.P$1
- new net N$117: D_P.CATHODE-, SW_P.P$1
- new net N$119: D_COLON.CATHODE-, SW_COLON.P$1
- new net N$12: IC1.PB2(MOSI), ICSP.4
- new net N$121: D_QM.CATHODE-, SW_QM.P$1
- new net N$125: D_MINUS.CATHODE-, SW_MINUS.P$1
- new net N$127: D_LCURL.CATHODE-, SW_LCURL.P$1
- new net N$129: D_QUOTE.CATHODE-, SW_QUOTE.P$1
- new net N$13: IC1.PB1(SCK), ICSP.3
- new net N$131: D_RSHIFT.CATHODE-, SW_RSHIFT.P$1
- new net N$135: D_PLUS.CATHODE-, SW_PLUS.P$1
- new net N$137: D_RCURL.CATHODE-, SW_RCURL.P$1
- new net N$139: D_ENTER.CATHODE-, SW_ENTER.P$1
- new net N$14: IC1.PE2/!HWB, R4.2, T3.P$1
- new net N$145: D_PIPE.CATHODE-, SW_PIPE.P$1
- new net N$147: D_BCK.CATHODE-, SW_BCK.P$1
- new net N$155: D_TILDE.CATHODE-, SW_TILDE.P$1
- new net N$17: D_TAB.CATHODE-, SW_TAB.P$1
- new net N$19: D_CAPS.CATHODE-, SW_CAPS.P$1
- new net N$2: J1.D-, R2.1
- new net N$20: D_LSHIFT.CATHODE-, SW_LSHIFT.P$1
- new net N$22: D_LCTRL.CATHODE-, SW_LCTRL.P$1
- new net N$25: D_1.CATHODE-, SW_1.P$1
- new net N$27: D_Q.CATHODE-, SW_Q.P$1
- new net N$29: D_A.CATHODE-, SW_A.P$1
- new net N$3: IC1.D+, R1.2
- new net N$31: D_Z.CATHODE-, SW_Z.P$1
- new net N$33: D_OS.CATHODE-, SW_OS.P$1
- new net N$35: D_2.CATHODE-, SW_2.P$1
- new net N$37: D_W.CATHODE-, SW_W.P$1
- new net N$39: D_S.CATHODE-, SW_S.P$1
- new net N$4: C4.1, IC1.XTAL2, X1.P$2
- new net N$41: D_X.CATHODE-, SW_X.P$1
- new net N$43: D_LALT.CATHODE-, SW_LALT.P$1
- new net N$45: D_3.CATHODE-, SW_3.P$1
- new net N$47: D_E.CATHODE-, SW_E.P$1
- new net N$49: D_D.CATHODE-, SW_D.P$1
- new net N$5: F1.1, J1.VBUS
- new net N$51: D_C.CATHODE-, SW_C.P$1
- new net N$53: D_SPACE.CATHODE-, SW_SPACE.P$1
- new net N$55: D_4.CATHODE-, SW_4.P$1
- new net N$57: D_R.CATHODE-, SW_R.P$1
- new net N$59: D_F.CATHODE-, SW_F.P$1
- new net N$61: D_V.CATHODE-, SW_V.P$1
- new net N$63: D_FN.CATHODE-, SW_FN.P$1
- new net N$65: D_5.CATHODE-, SW_5.P$1
- new net N$67: D_T.CATHODE-, SW_T.P$1
- new net N$69: D_G.CATHODE-, SW_G.P$1
- new net N$7: IC1.D-, R2.2
- new net N$71: D_B.CATHODE-, SW_B.P$1
- new net N$73: D_LA.CATHODE-, SW_LA.P$1
- new net N$75: D_6.CATHODE-, SW_6.P$1
- new net N$77: D_Y.CATHODE-, SW_Y.P$1
- new net N$79: D_H.CATHODE-, SW_H.P$1
- new net N$8: IC1.PB3(MISO), ICSP.5
- new net N$81: D_N.CATHODE-, SW_N.P$1
- new net N$83: D_UA.CATHODE-, SW_UA.P$1
- new net N$85: D_7.CATHODE-, SW_7.P$1
- new net N$87: D_U.CATHODE-, SW_U.P$1
- new net N$89: D_J.CATHODE-, SW_J.P$1
- new net N$9: C3.1, IC1.UCAP
- new net N$91: D_M.CATHODE-, SW_M.P$1
- new net N$93: D_DA.CATHODE-, SW_DA.P$1
- new net N$95: D_8.CATHODE-, SW_8.P$1
- new net N$97: D_I.CATHODE-, SW_I.P$1
- new net N$99: D_K.CATHODE-, SW_K.P$1
- new net RESET: IC1.!RESET, ICSP.6, R3.1, T1.P$1
- new net ROW1: IC1.PF1(ADC1), SW_0.P$2, SW_1.P$2, SW_2.P$2, SW_3.P$2, SW_4.P$2, SW_5.P$2, SW_6.P$2, SW_7.P$2, SW_8.P$2, SW_9.P$2, SW_ESC.P$2, SW_MINUS.P$2, SW_PIPE.P$2, SW_PLUS.P$2, SW_TILDE.P$2
- new net ROW2: IC1.PF4(ADC4), SW_BCK.P$2, SW_E.P$2, SW_I.P$2, SW_LCURL.P$2, SW_O.P$2, SW_P.P$2, SW_Q.P$2, SW_R.P$2, SW_RCURL.P$2, SW_T.P$2, SW_TAB.P$2, SW_U.P$2, SW_W.P$2, SW_Y.P$2
- new net ROW3: IC1.PD6(ADC9), SW_A.P$2, SW_CAPS.P$2, SW_COLON.P$2, SW_D.P$2, SW_ENTER.P$2, SW_F.P$2, SW_G.P$2, SW_H.P$2, SW_J.P$2, SW_K.P$2, SW_QUOTE.P$2, SW_S.P$2, S_L.P$2
- new net ROW4: IC1.PB4(ADC11), SW_B.P$2, SW_C.P$2, SW_GT.P$2, SW_LSHIFT.P$2, SW_LT.P$2, SW_M.P$2, SW_N.P$2, SW_QM.P$2, SW_RSHIFT.P$2, SW_V.P$2, SW_X.P$2, SW_Z.P$2
- new net ROW5: IC1.PB5(ADC12), SW_DA.P$2, SW_FN.P$2, SW_LA.P$2, SW_LALT.P$2, SW_LCTRL.P$2, SW_OS.P$2, SW_RA.P$2, SW_SPACE.P$2, SW_UA.P$2
- new net V+5: C1.1, C2.1, F1.2, IC1.AVCC@24, IC1.AVCC@44, IC1.UVCC, IC1.VBUS, IC1.VCC@14, IC1.VCC@34, ICSP.1, R3.2, R4.1
Other:
- moved on the sheet: IC1
